File: sesame.kicad_pcb (KiCad board)
At the start: 2 copper layers, 167 parts, among them U1 ATmega32A-PU

Commit message: Add files via upload
Parts:
- moved REF** 4.55 mm to (388.2, 176.0)
- moved REF** 4.42 mm to (261.5, 73.4)
- moved REF** 3.47 mm to (388.7, 76.3)
- moved R6 3.46 mm to (237.9, 77.9), turned to 350 degrees
- moved Reset1 3.30 mm to (245.2, 70.1), turned to 350 degrees
- moved Boot1 2.89 mm to (234.8, 68.2), turned to 350 degrees
- moved D69 1.95 mm to (369.3, 170.8)
- moved D68 1.93 mm to (350.3, 170.8)
- moved D70 1.91 mm to (388.4, 170.8)
- moved D16 1.44 mm to (375.2, 87.4)
- moved MX16 1.40 mm to (365.6, 83.7)
- moved REF** 0.97 mm to (193.4, 191.6)
- moved MX32 0.68 mm to (369.8, 102.7)
- moved D32 0.62 mm to (379.3, 106.6)
- moved D47 0.41 mm to (382.3, 125.6)
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Routing:
- net col15: track 218.9 -> 212.3 mm
- net Net-(D68-Pad2): track 6.10 -> 0.00 mm
- net row4: track 459.7 -> 454.5 mm
- net BOOT: track 77.3 -> 81.7 mm
- net +5V: track 143.6 -> 147.0 mm
- net RST: track 71.7 -> 75.0 mm
- net row3: track 395.6 -> 392.3 mm
- net Net-(D70-Pad2): track 5.86 -> 7.51 mm
- net row0: track 376.0 -> 377.6 mm
- net Net-(D69-Pad2): track 5.84 -> 7.31 mm
- net col17: track 250.5 -> 251.3 mm
- net row1: track 409.6 -> 410.2 mm

Commit message: Add files via upload
Routing:
- net Net-(D68-Pad2): track 0.00 -> 7.31 mm
- net row3: track 392.3 -> 395.6 mm

Commit message: Add files via upload
Parts:
- moved REF** 1.89 mm to (388.1, 74.5)
- moved REF** 0.76 mm to (24.5, 76.7)
- moved REF** 0.64 mm to (24.4, 174.4)
- moved REF** 0.25 mm to (388.0, 176.0)

Commit message: Add files via upload
Parts:
- added REF**: screw_hole, custom_parts:screw_hole, F.Cu at (193.5, 189.9)
- added REF**: screw_hole, custom_parts:screw_hole, F.Cu at (387.0, 153.2)
- moved REF** 106.4 mm to (281.6, 173.9)
- moved REF** 98.7 mm to (96.6, 172.5)
- moved REF** 2.33 mm to (25.3, 172.2)
- moved REF** 1.97 mm to (259.6, 73.9)
- moved AVR1 1.35 mm to (209.3, 65.4)
- moved C4 1.34 mm to (222.2, 83.8)
- moved C3 1.31 mm to (187.8, 86.8)
- moved XTAL1 1.28 mm to (221.0, 73.5)
- moved C2 1.27 mm to (192.9, 65.4)
- moved C5 1.27 mm to (222.2, 68.2)
- moved R1 1.27 mm to (153.5, 83.5)
- moved R2 1.27 mm to (153.6, 72.2)
- moved R3 1.27 mm to (153.6, 68.4)
- moved R4 1.27 mm to (153.5, 76.0)
- moved R5 1.27 mm to (153.5, 79.7)
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Routing:
- net col6: track 102.0 -> 105.6 mm
- net col10: track 108.1 -> 105.7 mm
- net col8: track 79.9 -> 78.3 mm
- net row4: track 454.5 -> 453.0 mm
- net Net-(D72-Pad1): track 34.9 -> 36.3 mm
- net Net-(D71-Pad1): track 39.0 -> 40.4 mm
- net col2: track 170.7 -> 171.9 mm
- net col5: track 115.0 -> 116.3 mm
- net col4: track 113.1 -> 114.4 mm
- net col0: track 202.3 -> 203.6 mm
- net Net-(R3-Pad1): track 12.5 -> 13.8 mm
- net Net-(R2-Pad1): track 8.73 -> 10.00 mm
- net col9: track 111.1 -> 109.9 mm
- net BOOT: track 81.7 -> 80.4 mm
- net col3: track 172.0 -> 173.2 mm
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
Commit message: Add files via upload
Other:
- board outline added: 370.3 x 130.8 mm

Commit message: Add files via upload
Parts:
- moved D17 1.72 mm to (46.0, 107.7)
- moved MX17 1.70 mm to (36.4, 104.0)
- moved D1 1.67 mm to (50.3, 88.6)
- moved MX1 1.53 mm to (40.8, 85.0)
- moved MX33 0.77 mm to (33.8, 123.1)
- moved D33 0.69 mm to (43.3, 126.9)
Routing:
- net row1: track 409.8 -> 411.7 mm
- net row0: track 378.4 -> 380.2 mm
- net Net-(D1-Pad2): track 7.94 -> 7.26 mm
