File: sesame.kicad_pcb (KiCad board)
At the start: 2 copper layers, 370.3 x 130.8 mm, 169 parts, among them U1 ATmega32A-PU

Commit message: Add files via upload
Routing:
- net col15: track 211.7 -> 217.5 mm
- net col11: track 142.5 -> 146.1 mm
- net col13: track 158.8 -> 161.5 mm
- net col2: track 171.9 -> 174.5 mm
- net col17: track 250.0 -> 251.6 mm
- net col16: track 242.3 -> 243.8 mm
- net col8: track 78.3 -> 79.7 mm
- net col0: track 204.1 -> 205.4 mm
- net row0: track 380.2 -> 378.9 mm
- net col14: track 133.3 -> 134.5 mm
- net row4: track 453.0 -> 454.0 mm
- net col1: track 219.8 -> 219.1 mm
- net col12: track 146.2 -> 146.9 mm

Commit message: Add files via upload
Parts:
- moved REF** 0.63 mm to (120.5, 75.9)

Commit message: Add files via upload
Parts:
- moved D65 1.93 mm to (186.2, 185.5)
- moved MX7 0.08 mm to (159.7, 98.1)
- moved MX20 0.06 mm to (109.1, 106.8)
- moved MX6 0.06 mm to (141.0, 94.1)
Routing:
- net Net-(D65-Pad2): track 8.13 -> 10.2 mm
- net row4: track 454.0 -> 452.6 mm
Changed lines of the file:
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@@
     (thickness 1.6)
     (drawings 22)
-    (tracks 830)
+    (tracks 831)
     (zones 0)
     (modules 169)
@@
   )
   (module MX_Alps_Hybrid:MX-1U-NoLED (layer F.Cu)
-    (at 178.2445 102.0572 348)
+    (at 178.27244 102.04196 348)
     (fp_text reference MX8 (at 0 3.175 168) (layer Dwgs.User)
       (effects (font (size 1 1) (thickness 0.15)))
@@
   )
   (module MX_Alps_Hybrid:MX-1.25U-NoLED (layer F.Cu)
-    (at 54.356 163.7284)
+    (at 54.31028 163.72332)
     (fp_text reference MX62 (at 0 3.175) (layer Dwgs.User)
       (effects (font (size 1 1) (thickness 0.15)))
@@
   )
   (module MX_Alps_Hybrid:MX-1.25U-NoLED (layer F.Cu)
-    (at 114.6937 166.4335 348)
+    (at 114.7064 166.4208 348)
     (fp_text reference MX63 (at 0 3.175 168) (layer Dwgs.User)
       (effects (font (size 1 1) (thickness 0.15)))
@@
   )
   (module MX_Alps_Hybrid:MX-2U-ReversedStabilizers-NoLED (layer F.Cu)
-    (at 144.9832 172.8597 348)
+    (at 144.99844 172.85716 348)
     (fp_text reference MX64 (at 0 3.175 168) (layer Dwgs.User)
       (effects (font (size 1 1) (thickness 0.15)))
@@
   )
   (module MX_Alps_Hybrid:MX-1.25U-NoLED (layer F.Cu)
-    (at 175.3108 179.3113 348)
+    (at 175.2854 179.30876 348)
     (fp_text reference MX65 (at 0 3.175 168) (layer Dwgs.User)
       (effects (font (size 1 1) (thickness 0.15)))
@@
   )
   (module MX_Alps_Hybrid:MX-1U-NoLED (layer F.Cu)
-    (at 165.0111 118.7323 348)
+    (at 165.0111 118.70944 348)
     (fp_text reference MX23 (at 0 3.175 168) (layer Dwgs.User)
       (effects (font (size 1 1) (thickness 0.15)))
@@
   )
   (module MX_Alps_Hybrid:MX-1U-NoLED (layer F.Cu)
-    (at 122.3518 90.1827 348)
+    (at 122.36196 90.1446 348)
     (fp_text reference MX5 (at 0 3.175 168) (layer Dwgs.User)
       (effects (font (size 1 1) (thickness 0.15)))
@@
   )
   (module MX_Alps_Hybrid:MX-1U-NoLED (layer F.Cu)
-    (at 109.0041 106.8197 348)
+    (at 109.0676 106.8324 348)
     (fp_text reference MX20 (at 0 3.175 168) (layer Dwgs.User)
       (effects (font (size 1 1) (thickness 0.15)))
@@
   )
   (module MX_Alps_Hybrid:MX-1U-NoLED (layer F.Cu)
-    (at 159.6009 98.0948 348)
+    (at 159.67964 98.0694 348)
     (fp_text reference MX7 (at 0 3.175 168) (layer Dwgs.User)
       (effects (font (size 1 1) (thickness 0.15)))
@@
   )
   (module MX_Alps_Hybrid:MX-1U-NoLED (layer F.Cu)
-    (at 140.9573 94.1197 348)
+    (at 141.01572 94.107 348)
     (fp_text reference MX6 (at 0 3.175 168) (layer Dwgs.User)
       (effects (font (size 1 1) (thickness 0.15)))
@@
   )
   (module Diode_THT:D_DO-35_SOD27_P7.62mm_Horizontal (layer F.Cu)
-    (at 184.2897 185.1787 78)
+    (at 186.182 185.547 78)
     (descr "Diode, DO-35_SOD27 series, Axial, Horizontal, pin pitch=7.62mm, , length*diameter=4*2mm^2, , http://www.diodes.com/_files/packages/DO-35.pdf")
     (tags "Diode DO-35_SOD27 series Axial Horizontal pin pitch 7.62mm  length 4mm diameter 2mm")
@@
   (segment (start 138.1379 177.2412) (end 133.7818 172.8851) (width 0.25) (layer F.Cu) (net 94))
   (segment (start 167.6019 185.1787) (end 162.8775 180.4543) (width 0.25) (layer F.Cu) (net 94))
-  (segment (start 184.2897 185.1787) (end 167.6019 185.1787) (width 0.25) (layer F.Cu) (net 94))
   (segment (start 270.0655 171.9072) (end 275.2344 166.7383) (width 0.25) (layer F.Cu) (net 94))
   (segment (start 251.9553 171.9072) (end 270.0655 171.9072) (width 0.25) (layer F.Cu) (net 94))
@@
   (segment (start 328.2823 166.7383) (end 275.2344 166.7383) (width 0.25) (layer F.Cu) (net 94))
   (segment (start 332.359 170.815) (end 328.2823 166.7383) (width 0.25) (layer F.Cu) (net 94))
-  (segment (start 210.058 178.816) (end 203.6953 185.1787) (width 0.25) (layer F.Cu) (net 94))
-  (segment (start 228.092 178.816) (end 210.058 178.816) (width 0.25) (layer F.Cu) (net 94))
-  (segment (start 203.6953 185.1787) (end 184.2897 185.1787) (width 0.25) (layer F.Cu) (net 94))
-  (segment (start 235.0008 171.9072) (end 228.092 178.816) (width 0.25) (layer F.Cu) (net 94))
-  (segment (start 251.9553 171.9072) (end 235.0008 171.9072) (width 0.25) (layer F.Cu) (net 94))
   (segment (start 193.59544 98.16835) (end 184.52381 89.09672) (width 0.25) (layer B.Cu) (net 94))
   (segment (start 193.59544 182.85796) (end 193.59544 98.16835) (width 0.25) (layer B.Cu) (net 94))
-  (segment (start 191.2747 185.1787) (end 193.59544 182.85796) (width 0.25) (layer B.Cu) (net 94))
-  (segment (start 184.2897 185.1787) (end 191.2747 185.1787) (width 0.25) (layer B.Cu) (net 94))
   (segment (start 184.52381 85.66234) (end 186.6138 83.57235) (width 0.25) (layer B.Cu) (net 94))
   (segment (start 184.52381 89.09672) (end 184.52381 85.66234) (width 0.25) (layer B.Cu) (net 94))
+  (segment (start 190.9064 185.547) (end 193.59544 182.85796) (width 0.25) (layer B.Cu) (net 94))
+  (segment (start 186.182 185.547) (end 190.9064 185.547) (width 0.25) (layer B.Cu) (net 94))
+  (segment (start 167.9702 185.547) (end 167.6019 185.1787) (width 0.25) (layer F.Cu) (net 94))
+  (segment (start 186.182 185.547) (end 167.9702 185.547) (width 0.25) (layer F.Cu) (net 94))
+  (segment (start 235.0008 171.9072) (end 251.9553 171.9072) (width 0.25) (layer F.Cu) (net 94))
+  (segment (start 228.092 178.816) (end 235.0008 171.9072) (width 0.25) (layer F.Cu) (net 94))
+  (segment (start 210.058 178.816) (end 228.092 178.816) (width 0.25) (layer F.Cu) (net 94))
+  (segment (start 203.327 185.547) (end 210.058 178.816) (width 0.25) (layer F.Cu) (net 94))
+  (segment (start 186.182 185.547) (end 203.327 185.547) (width 0.25) (layer F.Cu) (net 94))
   (segment (start 77.923 102.053) (end 78.6257 102.7557) (width 0.25) (layer F.Cu) (net 95))
   (segment (start 66.8255 102.053) (end 77.923 102.053) (width 0.25) (layer F.Cu) (net 95))
@@
   (segment (start 124.205687 162.551615) (end 127.085687 165.431615) (width 0.25) (layer F.Cu) (net 98))
   (segment (start 118.074672 162.551615) (end 124.205687 162.551615) (width 0.25) (layer F.Cu) (net 98))
-  (segment (start 183.578187 175.429415) (end 185.873987 177.725215) (width 0.25) (layer F.Cu) (net 99))
-  (segment (start 178.691772 175.429415) (end 183.578187 175.429415) (width 0.25) (layer F.Cu) (net 99))
+  (segment (start 181.355872 178.093515) (end 178.691772 175.429415) (width 0.25) (layer F.Cu) (net 99))
+  (segment (start 187.766287 178.093515) (end 181.355872 178.093515) (width 0.25) (layer F.Cu) (net 99))
   (segment (start 243.184918 75.8063) (end 244.455583 74.535635) (width 0.25) (layer B.Cu) (net 100))
   (segment (start 194.2338 68.33235) (end 201.70775 75.8063) (width 0.25) (layer B.Cu) (net 100))
